File: KICAD_DEV/USB-C-PD.kicad_sch (KiCad schematic)
At the start: 35 parts, among them J1 USB_C_Receptacle_USB2.0_14P, Q1 NMOS, U2 TPS26750, U3 TPD4S480

Commit message: pretty much done USB-PD wiring, just gotta do GPIO's
Parts:
- added C22: 10uF, symbol Device:C
- C14: value 10uF -> 0.1uF
Connections:
- net PP5V is gone; now on net VBUS: C19.1, C20.1, U2.28 (PP5V)
- net +3V3: now also C13.1; no longer C14.1
- net GND: now also C22.2
- net LDO_1V5: now also C12.1; no longer C13.1
- net LDO_3V3: now also C22.1; no longer C12.1
- net VBUS: no longer C1.1, C15.1, C16.1, C17.1, C18.1, C2.1, D1.2 (A), J1.A4 (VBUS), J1.A9 (VBUS), J1.B4 (VBUS), J1.B9 (VBUS), Q1.1 (D), U3.20 (VBUS)
- net VBUS_LV: now also C14.1
- new net VBUS_C: C1.1, C15.1, C16.1, C17.1, C18.1, C2.1, D1.2 (A), J1.A4 (VBUS), J1.A9 (VBUS), J1.B4 (VBUS), J1.B9 (VBUS), Q1.1 (D), U3.20 (VBUS)
- no-connect marks 4 -> 5
Other:
- moved on the sheet: C12, R3, R4, R5, R6

Commit message: cooking
Connections:
- net USB_D+: no longer U2.22 (USB_P)
- net USB_D-: no longer U2.23 (USB_N)
- no-connect marks 5 -> 14
Other:
- moved on the sheet: C1, C11, C12, C13, C14, C15, C16, C17, C18, C19, C2, C20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
