File: KICAD_DEV/the-secret-weapon.kicad_sch (KiCad schematic)
At the start: 0 parts

Commit message: added all 150 hierarchial sheets!
Other:
- added sheet 1 (1.kicad_sch)
- added sheet 10 (10.kicad_sch)
- added sheet 100 (100.kicad_sch)
- added sheet 101 (101.kicad_sch)
- added sheet 102 (102.kicad_sch)
- added sheet 103 (103.kicad_sch)
- added sheet 104 (104.kicad_sch)
- added sheet 105 (105.kicad_sch)
- added sheet 106 (106.kicad_sch)
- added sheet 107 (107.kicad_sch)
- added sheet 108 (108.kicad_sch)
- added sheet 109 (109.kicad_sch)
- added sheet 11 (11.kicad_sch)
- added sheet 110 (110.kicad_sch)
- added sheet 111 (111.kicad_sch)
- added sheet 112 (112.kicad_sch)
- added sheet 113 (113.kicad_sch)
- added sheet 114 (114.kicad_sch)
- added sheet 115 (115.kicad_sch)
- added sheet 116 (116.kicad_sch)
- added sheet 117 (117.kicad_sch)
- added sheet 118 (118.kicad_sch)
- added sheet 119 (119.kicad_sch)
- added sheet 12 (12.kicad_sch)
- added sheet 120 (120.kicad_sch)
- added sheet 121 (121.kicad_sch)
- added sheet 122 (122.kicad_sch)
- added sheet 123 (123.kicad_sch)
- added sheet 124 (124.kicad_sch)
- added sheet 125 (125.kicad_sch)
- added sheet 126 (126.kicad_sch)
- added sheet 127 (127.kicad_sch)
- added sheet 128 (128.kicad_sch)
- added sheet 129 (129.kicad_sch)
- added sheet 13 (13.kicad_sch)
- added sheet 130 (130.kicad_sch)
- added sheet 131 (131.kicad_sch)
- added sheet 132 (132.kicad_sch)
- added sheet 133 (133.kicad_sch)
- added sheet 134 (134.kicad_sch)
- added sheet 135 (135.kicad_sch)
- added sheet 136 (136.kicad_sch)
- added sheet 14 (14.kicad_sch)
- added sheet 15 (15.kicad_sch)
- added sheet 16 (16.kicad_sch)
- added sheet 17 (17.kicad_sch)
- added sheet 18 (18.kicad_sch)
- added sheet 19 (19.kicad_sch)
- added sheet 2 (2.kicad_sch)
- added sheet 20 (20.kicad_sch)
- added sheet 21 (21.kicad_sch)
- added sheet 22 (22.kicad_sch)
- added sheet 23 (23.kicad_sch)
- added sheet 24 (24.kicad_sch)
- added sheet 25 (25.kicad_sch)
- added sheet 26 (26.kicad_sch)
- added sheet 27 (27.kicad_sch)
- added sheet 28 (28.kicad_sch)
- added sheet 29 (29.kicad_sch)
- added sheet 3 (3.kicad_sch)
- added sheet 30 (30.kicad_sch)
- added sheet 31 (31.kicad_sch)
- added sheet 32 (32.kicad_sch)
- added sheet 33 (33.kicad_sch)
- added sheet 34 (34.kicad_sch)
- added sheet 35 (35.kicad_sch)
- added sheet 36 (36.kicad_sch)
- added sheet 37 (37.kicad_sch)
- added sheet 38 (38.kicad_sch)
- added sheet 39 (39.kicad_sch)
- added sheet 4 (4.kicad_sch)
- added sheet 40 (40.kicad_sch)
- added sheet 41 (41.kicad_sch)
- added sheet 42 (42.kicad_sch)
- added sheet 43 (43.kicad_sch)
- added sheet 44 (44.kicad_sch)
- added sheet 45 (45.kicad_sch)
- added sheet 46 (46.kicad_sch)
- added sheet 47 (47.kicad_sch)
- added sheet 48 (48.kicad_sch)
- added sheet 49 (49.kicad_sch)
- added sheet 5 (5.kicad_sch)
- added sheet 50 (50.kicad_sch)
- added sheet 51 (51.kicad_sch)
- added sheet 52 (52.kicad_sch)
- added sheet 53 (53.kicad_sch)
- added sheet 54 (54.kicad_sch)
- added sheet 55 (55.kicad_sch)
- added sheet 56 (56.kicad_sch)
- added sheet 57 (57.kicad_sch)
- added sheet 58 (58.kicad_sch)
- added sheet 59 (59.kicad_sch)
- added sheet 6 (6.kicad_sch)
- added sheet 60 (60.kicad_sch)
- added sheet 61 (61.kicad_sch)
- added sheet 62 (62.kicad_sch)
- added sheet 63 (63.kicad_sch)
- added sheet 64 (64.kicad_sch)
- added sheet 65 (65.kicad_sch)
- added sheet 66 (66.kicad_sch)
- added sheet 67 (67.kicad_sch)
- added sheet 68 (68.kicad_sch)
- added sheet 69 (69.kicad_sch)
- added sheet 7 (7.kicad_sch)
- added sheet 70 (70.kicad_sch)
- added sheet 71 (71.kicad_sch)
- added sheet 72 (72.kicad_sch)
- added sheet 73 (73.kicad_sch)
- added sheet 74 (74.kicad_sch)
- added sheet 75 (75.kicad_sch)
- added sheet 76 (76.kicad_sch)
- added sheet 77 (77.kicad_sch)
- added sheet 78 (78.kicad_sch)
- added sheet 79 (79.kicad_sch)
- added sheet 8 (8.kicad_sch)
- added sheet 80 (80.kicad_sch)
- added sheet 81 (81.kicad_sch)
- added sheet 82 (82.kicad_sch)
- added sheet 83 (83.kicad_sch)
- added sheet 84 (84.kicad_sch)
- added sheet 85 (85.kicad_sch)
- added sheet 86 (86.kicad_sch)
- added sheet 87 (87.kicad_sch)
- added sheet 88 (88.kicad_sch)
- added sheet 89 (89.kicad_sch)
- added sheet 9 (9.kicad_sch)
- added sheet 90 (90.kicad_sch)
- added sheet 91 (91.kicad_sch)
- added sheet 92 (92.kicad_sch)
- added sheet 93 (93.kicad_sch)
- added sheet 94 (94.kicad_sch)
- added sheet 95 (95.kicad_sch)
- added sheet 96 (96.kicad_sch)
- added sheet 97 (97.kicad_sch)
- added sheet 98 (98.kicad_sch)
- added sheet 99 (99.kicad_sch)

Commit message: adding some instructions inside of the schematic!
Other:
- sheet 1 renamed @KaiPereira - TMC2209 Motor Driver!
- note added: "Rename your page (not the file though please) with what your component is + your name by tapping "e" and changing the sheet name!"
- note added: "Select your page on the slack canvas!"
- note added: "Try not to modify this page so we don't get merge conflicts in the schematic editor!"
Changed lines of the file:
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@@
 	(generator_version "9.0")
 	(paper "A1")
+	(text "Select your page on the slack canvas!"
+		(exclude_from_sim no)
+		(at 430.53 -75.946 0)
+		(effects
+			(font
+				(size 5.08 5.08)
+			)
+		)
+	)
+	(text "Rename your page (not the file though please) with what your component is + your name by tapping \"e\" and changing the sheet name!"
+		(exclude_from_sim no)
+		(at 431.038 -37.846 0)
+		(effects
+			(font
+				(size 5.08 5.08)
+			)
+		)
+	)
+	(text "Try not to modify this page so we don't get merge conflicts in the schematic editor!"
+		(exclude_from_sim no)
+		(at 429.26 -93.726 0)
+		(effects
+			(font
+				(size 5.08 5.08)
+			)
+		)
+	)
 	(sheet
 		(at 478.79 189.23)
@@
 			(color 0 0 0 0.0000)
 		)
-		(property "Sheetname" "1"
+		(property "Sheetname" "@KaiPereira - TMC2209 Motor Driver!"
 			(at 149.86 20.8784 0)
 			(effects
