File: KICAD_DEV/the-secret-weapon.kicad_sch (KiCad schematic)
At the start: 0 parts

Commit message: wired my TMC2209 :D
Other:
- sheet @KaiPereira - TMC2209 Motor Driver! renamed @KaiPereira - TMC2209 Stepstick Motor Driver!
Changed lines of the file:
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@@
 			(color 0 0 0 0.0000)
 		)
-		(property "Sheetname" "@KaiPereira - TMC2209 Motor Driver!"
+		(property "Sheetname" "@KaiPereira - TMC2209 Stepstick Motor Driver!"
 			(at 149.86 20.8784 0)
 			(effects
