File: KICAD_DEV/brain-mcu.kicad_sch (KiCad schematic)
At the start: 22 parts, among them SW1 SW_Push, SW2 SW_Push, U1 STM32H743VITx, Y1 8 MHz, Y2 32.768 KHz

Commit message: finished routing my TMC2209 motor driver!
Connections:
- net TMC2209_DIAG: now also U1.29 (PA5); no longer U1.28 (PA4)
- net TMC2209_DIR: now also U1.32 (PC4); no longer U1.31 (PA7)
- net TMC2209_INDEX: now also U1.28 (PA4); no longer U1.29 (PA5)
- net TMC2209_RX: now also U1.23 (PA1); no longer U1.69 (PA10)
- net TMC2209_STEP: now also U1.31 (PA7); no longer U1.67 (PA8)
- net TMC2209_TX: now also U1.22 (PA0); no longer U1.68 (PA9)
Changed lines of the file:
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@@
+	(wire
+		(pts
+			(xy 247.65 100.33) (xy 245.11 100.33)
+		)
+		(stroke
+			(width 0)
+			(type default)
+		)
+	)
 	(wire
 		(pts
@@
 	(wire
 		(pts
+			(xy 247.65 194.31) (xy 245.11 194.31)
+		)
+		(stroke
+			(width 0)
+			(type default)
+		)
+	)
+	(wire
+		(pts
 			(xy 64.77 69.85) (xy 64.77 68.58)
 		)
@@
 	(wire
 		(pts
+			(xy 247.65 97.79) (xy 245.11 97.79)
+		)
+		(stroke
+			(width 0)
+			(type default)
+		)
+	)
+	(wire
+		(pts
 			(xy 68.58 209.55) (xy 78.74 209.55)
 		)
@@
 	(wire
 		(pts
-			(xy 247.65 123.19) (xy 245.11 123.19)
-		)
-		(stroke
-			(width 0)
-			(type default)
-		)
-	)
-	(wire
-		(pts
 			(xy 57.15 69.85) (xy 64.77 69.85)
 		)
@@
 	(wire
 		(pts
-			(xy 247.65 120.65) (xy 245.11 120.65)
-		)
-		(stroke
-			(width 0)
-			(type default)
-		)
-	)
-	(wire
-		(pts
 			(xy 95.25 69.85) (xy 95.25 68.58)
 		)
@@
 	(wire
 		(pts
-			(xy 247.65 118.11) (xy 245.11 118.11)
-		)
-		(stroke
-			(width 0)
-			(type default)
-		)
-	)
-	(wire
-		(pts
 			(xy 184.15 218.44) (xy 194.31 218.44)
 		)
@@
 			(width 0)
 			(type default)
-		)
-	)
-	(global_label "TMC2209_STEP"
-		(shape input)
-		(at 247.65 118.11 0)
-		(fields_autoplaced yes)
-		(effects
-			(font
-				(size 1.27 1.27)
-			)
-			(justify left)
-		)
-		(property "Intersheetrefs" "${INTERSHEET_REFS}"
-			(at 264.7259 118.11 0)
-			(effects
-				(font
-					(size 1.27 1.27)
-				)
-				(justify left)
-				(hide yes)
-			)
 		)
 	)
@@
 		)
 	)
+	(global_label "TMC2209_INDEX"
+		(shape input)
+		(at 247.65 107.95 0)
+		(fields_autoplaced yes)
+		(effects
+			(font
+				(size 1.27 1.27)
+			)
+			(justify left)
+		)
+		(property "Intersheetrefs" "${INTERSHEET_REFS}"
+			(at 265.6936 107.95 0)
+			(effects
+				(font
+					(size 1.27 1.27)
+				)
+				(justify left)
+				(hide yes)
+			)
+		)
+	)
 	(global_label "D-"
 		(shape input)
@@
 		)
 	)
-	(global_label "TMC2209_DIAG"
-		(shape input)
-		(at 247.65 107.95 0)
-		(fields_autoplaced yes)
-		(effects
-			(font
-				(size 1.27 1.27)
-			)
-			(justify left)
-		)
-		(property "Intersheetrefs" "${INTERSHEET_REFS}"
-			(at 264.3632 107.95 0)
-			(effects
-				(font
-					(size 1.27 1.27)
-				)
-				(justify left)
-				(hide yes)
-			)
-		)
-	)
 	(global_label "OSC32_OUT"
 		(shape output)
@@
 		)
 	)
+	(global_label "TMC2209_DIR"
+		(shape input)
+		(at 247.65 194.31 0)
+		(fields_autoplaced yes)
+		(effects
+			(font
+				(size 1.27 1.27)
+			)
+			(justify left)
+		)
+		(property "Intersheetrefs" "${INTERSHEET_REFS}"
+			(at 263.2746 194.31 0)
+			(effects
+				(font
+					(size 1.27 1.27)
+				)
+				(justify left)
+				(hide yes)
+			)
+		)
+	)
+	(global_label "TMC2209_STEP"
+		(shape input)
+		(at 247.65 115.57 0)
+		(fields_autoplaced yes)
+		(effects
+			(font
+				(size 1.27 1.27)
+			)
+			(justify left)
+		)
+		(property "Intersheetrefs" "${INTERSHEET_REFS}"
+			(at 264.7259 115.57 0)
+			(effects
+				(font
+					(size 1.27 1.27)
+				)
+				(justify left)
+				(hide yes)
+			)
+		)
+	)
 	(global_label "TMC2209_EN"
 		(shape input)
@@
 		(property "Intersheetrefs" "${INTERSHEET_REFS}"
 			(at 262.6093 113.03 0)
-			(effects
-				(font
-					(size 1.27 1.27)
-				)
-				(justify left)
-				(hide yes)
-			)
-		)
-	)
-	(global_label "TMC2209_TX"
-		(shape input)
-		(at 247.65 120.65 0)
-		(fields_autoplaced yes)
-		(effects
-			(font
-				(size 1.27 1.27)
-			)
-			(justify left)
-		)
-		(property "Intersheetrefs" "${INTERSHEET_REFS}"
-			(at 262.3069 120.65 0)
 			(effects
 				(font
@@
 		)
 	)
-	(global_label "TMC2209_DIR"
-		(shape input)
-		(at 247.65 115.57 0)
-		(fields_autoplaced yes)
-		(effects
-			(font
-				(size 1.27 1.27)
-			)
-			(justify left)
-		)
-		(property "Intersheetrefs" "${INTERSHEET_REFS}"
-			(at 263.2746 115.57 0)
-			(effects
-				(font
-					(size 1.27 1.27)
-				)
-				(justify left)
-				(hide yes)
-			)
-		)
-	)
-	(global_label "TMC2209_INDEX"
+	(global_label "TMC2209_TX"
+		(shape input)
+		(at 247.65 97.79 0)
+		(fields_autoplaced yes)
+		(effects
+			(font
+				(size 1.27 1.27)
+			)
+			(justify left)
+		)
+		(property "Intersheetrefs" "${INTERSHEET_REFS}"
+			(at 262.3069 97.79 0)
+			(effects
+				(font
+					(size 1.27 1.27)
+				)
+				(justify left)
+				(hide yes)
+			)
+		)
+	)
+	(global_label "TMC2209_DIAG"
 		(shape input)
 		(at 247.65 110.49 0)
@@
 		)
 		(property "Intersheetrefs" "${INTERSHEET_REFS}"
-			(at 265.6936 110.49 0)
+			(at 264.3632 110.49 0)
 			(effects
 				(font
@@
 	(global_label "TMC2209_RX"
 		(shape input)
-		(at 247.65 123.19 0)
-		(fields_autoplaced yes)
-		(effects
-			(font
-				(size 1.27 1.27)
-			)
-			(justify left)
-		)
-		(property "Intersheetrefs" "${INTERSHEET_REFS}"
-			(at 262.6093 123.19 0)
-			(effects
-				(font
+		(at 247.65 100.33 0)
+		(fields_autoplaced yes)
+		(effects
+			(font
+				(size 1.27 1.27)
+			)
+			(justify left)
+		)
+		(property "Intersheetrefs" "${INTERSHEET_REFS}"
+			(at 262.6093 100.33 0)
+			(effects
+				(font
