File: KICAD_DEV/2.kicad_sch (KiCad schematic)
At the start: 0 parts

Commit message: testing
Parts:
- added C18: 0.1uF, Capacitor_SMD:C_0402_1005Metric, symbol Device:C
- added J3: Conn_01x05, Connector_JST:JST_XH_B5B-XH-AM_1x05_P2.50mm_Vertical, symbol Connector_Generic:Conn_01x05
- added R5: 1K, Resistor_SMD:R_0402_1005Metric, symbol Device:R
Connections:
- new net: J3.5 (Pin_5), R5.1
- new net +5V: C18.1, J3.2 (Pin_2)
- new net GND: C18.2, J3.1 (Pin_1)
- new net TFT_NRST: R5.2
- new net TFT_RX: J3.4 (Pin_4)
- new net TFT_TX: J3.3 (Pin_3)
